File: laserDriverButterfly_V2/Mezonin/Mezonin/Mezonin.sch (KiCad schematic (older format))
At the start: 12 parts, among them U1 LD

Commit message: update mez
Parts:
- U1: symbol aab_lib:LD -> Mezonin-rescue:LD-aab_lib
Changed lines of the file:
@@
 $EndDescr
 $Comp
-L aab_lib:LD U1
+L Mezonin-rescue:LD-aab_lib U1
 U 1 1 6192372B
 P 5250 2700
