File: laserDriverButterfly_V2/Motherboard/Motherboard.sch (KiCad schematic (older format))
At the start: 41 parts, among them CON1 Barrel_Jack_Switch, U1 LM317_3PinPackage, X1 Conn_Coaxial

Commit message: update voltreg and motherboard
Parts:
- VR1: symbol aab_lib:3266W-1-102LF -> Motherboard-rescue:3266W-1-102LF-aab_lib
Other:
- moved on the sheet: BUSIN1, BUSIN2, BUSIN3, BUSIN4, BUSLD1, BUSLD2, BUSLD3, BUSLD4, BUSOUT1, BUSOUT2, BUSOUT3, BUSOUT4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
