File: laserDriverButterfly_V2/VoltageRegulator/VoltReg.sch (KiCad schematic (older format))
At the start: 22 parts, among them U1 LM317_3PinPackage, U2 IRF5852PbF, U3 LP3878MR-ADJ_NOPB

Commit message: update voltreg and motherboard
Parts:
- U2: symbol aab_lib:IRF5852PbF -> VoltReg-rescue:IRF5852PbF-aab_lib
- U3: symbol aab_lib:LP3878MR-ADJ_NOPB -> VoltReg-rescue:LP3878MR-ADJ_NOPB-aab_lib
- VR1, VR2: symbol aab_lib:3266W-1-102LF -> VoltReg-rescue:3266W-1-102LF-aab_lib
Changed lines of the file:
@@
 	3950 2650 3950 2700
 $Comp
-L aab_lib:3266W-1-102LF VR?
+L VoltReg-rescue:3266W-1-102LF-aab_lib VR?
 U 1 1 62062E8C
 P 4200 2900
@@
 $EndComp
 $Comp
-L aab_lib:3266W-1-102LF VR?
+L VoltReg-rescue:3266W-1-102LF-aab_lib VR?
 U 1 1 62062EC3
 P 3950 4850
@@
 $EndComp
 $Comp
-L aab_lib:LP3878MR-ADJ_NOPB U?
+L VoltReg-rescue:LP3878MR-ADJ_NOPB-aab_lib U?
 U 1 1 62062EEA
 P 3550 4100
@@
 $EndComp
 $Comp
-L aab_lib:IRF5852PbF U?
+L VoltReg-rescue:IRF5852PbF-aab_lib U?
 U 1 1 62062F0F
 P 5850 3300
